Commit message: aaa

File: src/robot_description/urdf/robot_description.urdf (robot description, URDF)
Before this commit: robot robot_description, 11 links, 10 joints
Links:
- link base_link: mass 7.14346940014238 -> 4.69019425963942
- link link1: mass 0.669152126885544 -> 0.254561487975799
- link link2: mass 0.245621615505831 -> 1.04400658098434
- link link3: mass 0.149633690086611 -> 0.360136694535127
- link link4: mass 0.124846801253627 -> 0.45505308641721
- link link5: mass 0.0454906138754859 -> 0.191964378686302
- link link6: mass 0.0271812481344181 -> 0.00925955650346606
- link link_hand: mass 0.159305199837658 -> 0.0391687383342846
- link link_left: mass 0.00926377813438083 -> 0.0102982298696928
- link link_right: mass 0.0092637781343808 -> 0.0102982312448067
Joints:
- joint joint1: axis 0 0 1 -> 0 0 -1; limit lower=-3.14 upper=1 effort=100 velocity=1 -> lower=-3.14 upper=3.14 effort=100 velocity=1
- joint joint2: axis 0 0 -1 -> 0 0 1; limit lower=-3.14 upper=0.8 effort=100 velocity=1 -> lower=-3.14 upper=3.14 effort=100 velocity=1; origin xyz=0 0 0.1287 rpy=1.5707963267949 0 0 -> xyz=0.0600000000000005 0 0.0780000000000011 rpy=1.5707963267949 0 0
- joint joint3: limit lower=-3.14 upper=0.6 effort=100 velocity=1 -> lower=-3.14 upper=3.14 effort=100 velocity=1; origin xyz=0 0.22 0 rpy=0 0 1.5707963267949 -> xyz=0 0.179999999999999 0 rpy=0 0 1.5707963267949
- joint joint4: limit lower=-3.14 upper=0.785 effort=100 velocity=1 -> lower=-3.14 upper=3.14 effort=100 velocity=1; origin xyz=0 0 0 rpy=1.5707963267949 0 0 -> xyz=0.0599997753303093 0 0 rpy=1.5707963267949 0 -0.00011195880316143
- joint joint5: limit lower=-3.14 upper=0.785 effort=100 velocity=1 -> lower=-3.14 upper=3.14 effort=100 velocity=1; origin xyz=0 0 0.168499999999998 rpy=1.57079632679489 0 3.14159265358979 -> xyz=1.71296968475843E-05 0 0.150993281525449 rpy=1.5707963267949 0 -3.14159265358979
- joint joint6: origin xyz=0 0 0 rpy=1.57079632679489 0 -1.5707963267949 -> xyz=0 0 0 rpy=1.5707963267949 0 1.57090828559806
- joint joint_hand: limit lower=-3.14 upper=3.14 effort=0 velocity=0 -> lower=-3.14 upper=3.14 effort=100 velocity=1; origin xyz=0 0 -0.0934999999999999 rpy=1.5707963267949 0 -1.5707963267949 -> xyz=-0.307999999999998 0 0.318 rpy=-1.5707963267949 0 1.5707963267949
- joint joint_left: limit lower=-0.01 upper=0.01 effort=100 velocity=1 -> lower=0 upper=0.05 effort=100 velocity=1; mimic (none) -> joint=joint_right multiplier=-1 offset=0; origin xyz=0 -0.04 0 rpy=0 0 1.5707963267949 -> xyz=0 0.204632399732943 -0.307999999999999 rpy=1.5707963267949 -1.5707963267949 0
- joint joint_right: limit lower=-0.01 upper=0.01 effort=100 velocity=1 -> lower=0 upper=0.05 effort=100 velocity=1; origin xyz=0 -0.04 0 rpy=0 0 -1.5707963267949 -> xyz=0 0.204632399732943 -0.307999999999999 rpy=1.5707963267949 1.5707963267949 0
